File: _saved_pantry_monitor.sch (KiCad schematic (older format))
At the start: 38 parts, among them J1 raspi vcc/gnd, J10 LED 4, J11 Switch 4, J12 LED 5, J13 Switch 5, J2 LED input, J3 Switch output, J4 LED 1, J5 Switch 1, J6 LED 2, J7 Switch 2, J8 LED 3, J9 Switch 3, Q1 Q_NPN_BEC, Q2 Q_NPN_BEC, Q3 Q_NPN_BEC, Q4 Q_NPN_BEC, Q5 Q_NPN_BEC

Commit message: First mostly functional version of board.
Parts:
- removed Q1, Q2, Q3, Q4, Q5: Q_NPN_BEC, symbol Q_NPN_BEC
- added Q1, Q2, Q3, Q4, Q5: 2N3904, TO_SOT_Packages_THT:TO-92_Inline_Narrow_Oval, symbol 2N3904
- J1, J10, J11, J12, J13, J4, J5, J6, J7, J8, J9: footprint (none) -> Pin_Headers:Pin_Header_Straight_1x02_Pitch2.54mm
- J2, J3: footprint (none) -> Pin_Headers:Pin_Header_Straight_1x05_Pitch2.54mm
- R1, R10, R11, R12, R13, R14, R15, R16, R17, R18, R19, R2, R20, R4, R5, R6, R7, R8, R9: footprint (none) -> Resistors_THT:R_Axial_DIN0204_L3.6mm_D1.6mm_P7.62mm_Horizontal
- R3: value R -> 330; footprint (none) -> Resistors_THT:R_Axial_DIN0204_L3.6mm_D1.6mm_P7.62mm_Horizontal
Connections:
- wire segments 99 -> 94
