File: pantry_monitor.sch (KiCad schematic (older format))
At the start: 25 parts

Commit message: Initial commit.
Parts:
- removed J?: switch 1, symbol CONN_01X02
- removed R?: R, symbol R
- added J11: Switch 4, symbol CONN_01X02
- added J13: Switch 5, symbol CONN_01X02
- added J5: Switch 1, symbol CONN_01X02
- added J7: Switch 2, symbol CONN_01X02
- added J9: Switch 3, symbol CONN_01X02
- added R11, R15, R19, R7: 330, symbol R
- added R12, R16, R20, R4, R8: 1k, symbol R
- added R3: R, symbol R
- gave numbers to parts that had none: 23
Connections:
- net GND: now also R12.2, R16.2, R20.2, R4.2, R8.2
- net VCC: now also R11.1, R15.1, R19.1, R3.1, R7.1
- removed net Label1: J3.1 (P1), J3.2 (P2), J3.3 (P3), J3.4 (P4), J3.5 (P5)
- new net: J5.1 (P1), R3.2
- new net: J7.1 (P1), R7.2
- new net: J9.1 (P1), R11.2
- new net: J11.1 (P1), R15.2
- new net: J13.1 (P1), R19.2
- new net Switch1: J3.1 (P1), J5.2 (P2), R4.1
- new net Switch2: J3.2 (P2), J7.2 (P2), R8.1
- new net Switch3: J3.3 (P3), J9.2 (P2), R12.1
- new net Switch4: J11.2 (P2), J3.4 (P4), R16.1
- new net Switch5: J13.2 (P2), J3.5 (P5), R20.1
Other:
- moved on the sheet: J1, J3

Commit message: First mostly functional version of board.
Parts:
- J1, J10, J11, J12, J13, J4, J5, J6, J7, J8, J9: footprint (none) -> Pin_Headers:Pin_Header_Straight_1x02_Pitch2.54mm
- J2, J3: footprint (none) -> Pin_Headers:Pin_Header_Straight_1x05_Pitch2.54mm
- Q1, Q2, Q3, Q4, Q5: footprint (none) -> TO_SOT_Packages_THT:TO-92_Inline_Narrow_Oval
- R1, R10, R11, R12, R13, R14, R15, R16, R17, R18, R19, R2, R20, R4, R5, R6, R7, R8, R9: footprint (none) -> Resistors_THT:R_Axial_DIN0204_L3.6mm_D1.6mm_P7.62mm_Horizontal
- R3: value R -> 330; footprint (none) -> Resistors_THT:R_Axial_DIN0204_L3.6mm_D1.6mm_P7.62mm_Horizontal
